File: sheets/storage.kicad_sch (KiCad schematic)
At the start: 5 parts, among them U6 W25Q128JVPIQ

Commit message: Populate U6 flash, add silkscreen section labels, design brief
U6 and its passives are now fitted (BOM 24 lines / 43 parts). Top silk names each section; cell outline on the back. docs/designBrief.html generated. ERC and DRC unchanged: 0 errors. Firmware does not use U6 yet.

Co-Authored-By: Claude Opus 5.5 <noreply@anthropic.com>
Parts:
- C12, R16, R18, R19, U6: now fitted; now in the parts list
Other:
- note added: "U6 16 MB NOR on SPI2 for clip storage (about 33 min of audio on top of the module's own flash)"
- note removed: "U6 optional 16 MB NOR on SPI2 (FSPI pins). NOT FITTED by default: clips live on the module's 8 MB flash"
- title: smart-bookmark-esp32s3 - Optional external SPI flash (DNP) -> smart-bookmark-esp32s3 - External 16 MB SPI flash for clips
Changed lines of the file:
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@@
 	(generator_version "10.0")
 	(paper "A4")
-	(title_block (title "smart-bookmark-esp32s3 - Optional external SPI flash (DNP)") (date "2026-10-05") (rev "A") (company "Smart bookmark voice recorder"))
+	(title_block (title "smart-bookmark-esp32s3 - External 16 MB SPI flash for clips") (date "2026-10-05") (rev "A") (company "Smart bookmark voice recorder"))
 	(rectangle (start 60.96 55.88) (end 248.92 149.86) (stroke (width 0.2) (type dash)) (fill (type none)))
-	(text "U6 optional 16 MB NOR on SPI2 (FSPI pins). NOT FITTED by default: clips live on the module's 8 MB flash" (exclude_from_sim no) (at 62.23 54.61 0) (effects (font (size 1.5 1.5)) (justify left bottom)))
+	(text "U6 16 MB NOR on SPI2 for clip storage (about 33 min of audio on top of the module's own flash)" (exclude_from_sim no) (at 62.23 54.61 0) (effects (font (size 1.5 1.5)) (justify left bottom)))
 	(symbol (lib_id "Memory_Flash:W25Q128JVP") (at 149.86 101.6 0) (unit 1) (body_style 1)
-		(exclude_from_sim no) (in_bom no) (on_board yes) (in_pos_files no) (dnp yes)
+		(exclude_from_sim no) (in_bom yes) (on_board yes) (in_pos_files yes) (dnp no)
 		(property "Reference" "U6" (at 149.86 85.09 0) (show_name no) (do_not_autoplace no) (effects (font (size 1.27 1.27))))
 		(property "Value" "W25Q128JVPIQ" (at 149.86 118.11 0) (show_name no) (do_not_autoplace no) (effects (font (size 1.27 1.27))))
@@
 	)
 	(symbol (lib_id "Device:C") (at 205.74 101.6 0) (unit 1) (body_style 1)
-		(exclude_from_sim no) (in_bom no) (on_board yes) (in_pos_files no) (dnp yes)
+		(exclude_from_sim no) (in_bom yes) (on_board yes) (in_pos_files yes) (dnp no)
 		(property "Reference" "C12" (at 208.28 100.33 0) (show_name no) (do_not_autoplace no) (effects (font (size 1.27 1.27)) (justify left)))
 		(property "Value" "100nF" (at 208.28 102.87 0) (show_name no) (do_not_autoplace no) (effects (font (size 1.27 1.27)) (justify left)))
@@
 	)
 	(symbol (lib_id "Device:R") (at 226.06 101.6 0) (unit 1) (body_style 1)
-		(exclude_from_sim no) (in_bom no) (on_board yes) (in_pos_files no) (dnp yes)
+		(exclude_from_sim no) (in_bom yes) (on_board yes) (in_pos_files yes) (dnp no)
 		(property "Reference" "R16" (at 228.6 100.33 0) (show_name no) (do_not_autoplace no) (effects (font (size 1.27 1.27)) (justify left)))
 		(property "Value" "100k" (at 228.6 102.87 0) (show_name no) (do_not_autoplace no) (effects (font (size 1.27 1.27)) (justify left)))
@@
 	(hierarchical_label "FLASH_CS" (shape bidirectional) (at 226.06 107.95 270) (effects (font (size 1.27 1.27)) (justify right)))
 	(symbol (lib_id "Device:R") (at 86.36 124.46 0) (unit 1) (body_style 1)
-		(exclude_from_sim no) (in_bom no) (on_board yes) (in_pos_files no) (dnp yes)
+		(exclude_from_sim no) (in_bom yes) (on_board yes) (in_pos_files yes) (dnp no)
 		(property "Reference" "R18" (at 88.9 123.19 0) (show_name no) (do_not_autoplace no) (effects (font (size 1.27 1.27)) (justify left)))
 		(property "Value" "10k" (at 88.9 125.73 0) (show_name no) (do_not_autoplace no) (effects (font (size 1.27 1.27)) (justify left)))
@@
 	(label "FLASH_WP" (at 86.36 130.81 270) (effects (font (size 1.27 1.27)) (justify right bottom)))
 	(symbol (lib_id "Device:R") (at 104.14 124.46 0) (unit 1) (body_style 1)
-		(exclude_from_sim no) (in_bom no) (on_board yes) (in_pos_files no) (dnp yes)
+		(exclude_from_sim no) (in_bom yes) (on_board yes) (in_pos_files yes) (dnp no)
 		(property "Reference" "R19" (at 106.68 123.19 0) (show_name no) (do_not_autoplace no) (effects (font (size 1.27 1.27)) (justify left)))
 		(property "Value" "10k" (at 106.68 125.73 0) (show_name no) (do_not_autoplace no) (effects (font (size 1.27 1.27)) (justify left)))
